File: BLESEN.kicad_pcb (KiCad board)
At the start: 4 copper layers, 35 x 25 mm, 41 parts, among them J1 Conn_ARM_SWD_TagConnect_TC2030, J2 Conn_01x04_Pin, J3 Conn_01x04_Pin, Q1 Q_Photo_NPN, U1 STM32WB55CGUx, U2 SHTC3, Y1 32 Mhz, Y2 Crystal

Commit message: Tweaks
Parts:
- added FID1: Fiducial, Fiducial:Fiducial_0.5mm_Mask1mm, F.Cu at (152.0, 78.0)
- added FID2: Fiducial, Fiducial:Fiducial_0.5mm_Mask1mm, F.Cu at (131.0, 78.0)
- added FID3: Fiducial, Fiducial:Fiducial_0.5mm_Mask1mm, F.Cu at (152.0, 98.0)
- J2, J3: value Conn_01x04_Pin -> ~
- Y1: value 32 Mhz -> 32 MHz
- Y2: value Crystal -> 32.768KHz
Connections:
- net /OSC_IN renamed /OSC_HSE_IN
- net /OSC_OUT renamed /OSC_HSE_OUT
- net /SWDCLK renamed SWDCLK
- net /SWDIO renamed SWDIO
- net Net-(U1-PC14) renamed /OSC_LSE_IN
- net Net-(U1-PC15) renamed /OSC_LSE_OUT
Routing:
- net GND: vias 86 -> 88
Other:
- board text added: "3.3V"
- board text added: "URX"
- board text added: "UTX"
