File: BLESEN.kicad_pcb (KiCad board)
At the start: 4 copper layers, 37.6 x 25 mm, 43 parts, among them J1 Conn_ARM_SWD_TagConnect_TC2030, Q1 Q_Photo_NPN, U1 STM32WB55CGUx, U2 SHTC3, Y1 32 MHz, Y2 32.768KHz

Commit message: Release 0.4
Parts:
- U2: value SHTC3 -> SHT4x; footprint Sensor_Humidity:Sensirion_DFN-4-1EP_2x2mm_P1mm_EP0.7x1.6mm -> Sensor_Humidity:Sensirion_DFN-4_1.5x1.5mm_P0.8mm_SHT4x_NoCentralPad
- moved FID1 27.7 mm to (152.0, 101.0)
- moved FID2 11.3 mm to (129.0, 101.0)
- moved R2 5.04 mm to (135.4, 87.5), turned to -90 degrees
- moved C12 2.57 mm to (130.8, 88.6), turned to -90 degrees
- moved R1 2.14 mm to (135.4, 89.7)
- moved R3 0.60 mm to (151.6, 99.0)
- moved U2 0.10 mm to (132.8, 88.6), turned to 180 degrees
Connections:
- U2 pad 1: +3.3V -> SDA
- U2 pad 3: SDA -> +3.3V
Routing:
- net SCL: track 17.3 -> 8.40 mm
- net GND: track 12.7 -> 10.3 mm, vias 100 -> 98
- net +3.3V: track 67.1 -> 68.2 mm
- net SDA: track 9.15 -> 8.15 mm
- net LED: track 10.6 -> 10.0 mm
Other:
- board text added: "0.4"
- board text removed: "0.3"
