File: BLESEN.kicad_sch (KiCad schematic)
At the start: 41 parts, among them J1 Conn_ARM_SWD_TagConnect_TC2030, J2 Conn_01x04_Pin, J3 Conn_01x04_Pin, Q1 Q_Photo_NPN, U1 STM32WB55CGUx, U2 SHTC3, Y1 32 Mhz, Y2 Crystal

Commit message: Tweaks
Parts:
- added FID1, FID2, FID3: Fiducial, Fiducial:Fiducial_0.5mm_Mask1mm, symbol Mechanical:Fiducial
- AE1: symbol Device:Antenna -> Device:Antenna_Shield
- J2, J3: value Conn_01x04_Pin -> ~
- Y1: value 32 Mhz -> 32 MHz; LCSC C113671 -> C843260
- Y2: value Crystal -> 32.768KHz
Connections:
- net GND: now also AE1.2 (Shield)
- net OSC_LSE_OUT: now reaches C15.1, U1.3 (PC15), Y2.2
- net OSC_LSE_IN: now reaches C14.1, U1.2 (PC14), Y2.1
- net OSC_IN renamed OSC_HSE_IN
- net OSC_OUT renamed OSC_HSE_OUT
Other:
- note added: "Fiducial Marker"
- note added: "UART Connector"
- moved on the sheet: C14, C15, J3, Y2
