File: BLESEN.kicad_sch (KiCad schematic)
At the start: 43 parts, among them J1 Conn_ARM_SWD_TagConnect_TC2030, Q1 Q_Photo_NPN, U1 STM32WB55CGUx, U2 SHTC3, Y1 32 MHz, Y2 32.768KHz

Commit message: Release 0.4
Parts:
- C10: LCSC C1525 -> C1546
- U2: value SHTC3 -> SHT4x; footprint Sensor_Humidity:Sensirion_DFN-4-1EP_2x2mm_P1mm_EP0.7x1.6mm -> Sensor_Humidity:Sensirion_DFN-4_1.5x1.5mm_P0.8mm_SHT4x_NoCentralPad; symbol Sensor_Humidity:SHTC3 -> Sensor_Humidity:SHT4x
Connections:
- net +3.3V: now also U2.3 (VDD); no longer U2.1 (VDD)
- net SDA: now also U2.1 (SDA); no longer U2.3 (SDA)
Changed lines of the file:
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@@
 			)
 		)
-		(property "LCSC" "C1525"
+		(property "LCSC" "C1546"
 			(at 180.848 24.384 0)
 			(effects
@@
 	)
 	(symbol
-		(lib_id "Sensor_Humidity:SHTC3")
+		(lib_id "Sensor_Humidity:SHT4x")
 		(at 38.1 124.46 180)
 		(unit 1)
@@
 			)
 		)
-		(property "Value" "SHTC3"
+		(property "Value" "SHT4x"
 			(at 31.75 125.7299 0)
 			(effects
@@
 			)
 		)
-		(property "Footprint" "Sensor_Humidity:Sensirion_DFN-4-1EP_2x2mm_P1mm_EP0.7x1.6mm"
-			(at 33.02 115.57 0)
+		(property "Footprint" "Sensor_Humidity:Sensirion_DFN-4_1.5x1.5mm_P0.8mm_SHT4x_NoCentralPad"
+			(at 34.29 118.11 0)
 			(effects
 				(font
 					(size 1.27 1.27)
 				)
+				(justify left)
 				(hide yes)
 			)
 		)
-		(property "Datasheet" "https://www.sensirion.com/fileadmin/user_upload/customers/sensirion/Dokumente/0_Datasheets/Humidity/Sensirion_Humidity_Sensors_SHTC3_Datasheet.pdf"
-			(at 45.72 135.89 0)
+		(property "Datasheet" "https://sensirion.com/media/documents/33FD6951/624C4357/Datasheet_SHT4x.pdf"
+			(at 34.29 115.57 0)
 			(effects
 				(font
 					(size 1.27 1.27)
 				)
+				(justify left)
 				(hide yes)
 			)
 		)
-		(property "Description" "Humidity and Temperature Sensor, +/-2%RH, +/-0.2degC, I2C, 1.62-3.6V, DFN-4"
+		(property "Description" "Digital Humidity and Temperature Sensor, +/-1%RH, +/-0.1degC, I2C, 1.08-3.6V, 16bit, DFN-4"
 			(at 38.1 124.46 0)
 			(effects
@@
 		(pin "3"
 		)
-		(pin "5"
-		)
 		(pin "2"
