File: BLESEN_Panelized.kicad_pcb (KiCad board)
At the start: 4 copper layers, 92.2 x 95 mm, 264 parts, among them J1 Conn_ARM_SWD_TagConnect_TC2030, Q1 Q_Photo_NPN, U1 STM32WB55CGUx, U2 SHTC3, Y1 32 MHz, Y2 32.768KHz

Commit message: Release 0.4
Parts:
- removed the AE1 at (180.8, 34.9)
- removed the AE1 at (140.2, 34.9)
- removed the AE1 at (180.8, 62.9)
- removed the AE1 at (180.8, 90.9)
- removed the AE1 at (140.2, 90.9)
- removed the AE1 at (140.2, 62.9)
- removed the BT1 at (165.9, 95.6)
- removed the BT1 at (125.3, 67.6)
- removed the BT1 at (165.9, 67.6)
- removed the BT1 at (125.3, 39.6)
- removed the BT1 at (165.9, 39.6)
- removed the BT1 at (125.3, 95.6)
- removed the C1 at (161.2, 70.2)
- removed the C1 at (120.5, 98.2)
- removed the C1 at (161.2, 98.2)
- removed the C1 at (161.2, 42.1)
- removed the C1 at (120.5, 42.1)
- removed the C1 at (120.5, 70.2)
- removed the C10 at (170.9, 91.5)
- removed the C10 at (130.3, 63.5)
- removed the C10 at (130.3, 35.5)
- removed the C10 at (130.3, 91.5)
- removed the C10 at (170.9, 63.5)
- removed the C10 at (170.9, 35.5)
- removed the C11 at (171.9, 35.5)
- removed the C11 at (171.9, 91.5)
- removed the C11 at (171.9, 63.5)
- removed the C11 at (131.3, 91.5)
- removed the C11 at (131.3, 35.5)
- removed the C11 at (131.3, 63.5)
- removed the C12 at (114.1, 36.9)
- removed the C12 at (114.1, 92.9)
- removed the C12 at (154.7, 92.9)
- removed the C12 at (154.7, 64.9)
- removed the C12 at (154.7, 36.9)
- removed the C12 at (114.1, 64.9)
- removed the C13 at (127.6, 100.7)
- removed the C13 at (168.2, 72.7)
- removed the C13 at (127.6, 72.7)
- removed the C13 at (127.6, 44.7)
- removed the C13 at (168.2, 100.7)
- removed the C13 at (168.2, 44.7)
- removed the C14 at (164.1, 73.8)
- removed the C14 at (123.5, 101.8)
- removed the C14 at (164.1, 101.8)
- removed the C14 at (164.1, 45.8)
- removed the C14 at (123.5, 73.8)
- removed the C14 at (123.5, 45.8)
- removed the C15 at (166.4, 45.8)
- removed the C15 at (125.8, 101.8)
- removed the C15 at (125.8, 73.8)
- removed the C15 at (125.8, 45.8)
- removed the C15 at (166.4, 73.8)
- removed the C15 at (166.4, 101.8)
- removed the C16 at (126.4, 61.7)
- removed the C16 at (126.4, 89.7)
- removed the C16 at (167.0, 89.7)
- removed the C16 at (167.0, 61.7)
- removed the C16 at (167.0, 33.7)
- removed the C16 at (126.4, 33.7)
- removed the C17 at (162.5, 33.1)
- removed the C17 at (162.5, 89.1)
- removed the C17 at (121.9, 33.1)
- removed the C17 at (121.9, 89.1)
- removed the C17 at (121.9, 61.1)
- removed the C17 at (162.5, 61.1)
- removed the C18 at (162.2, 87.8)
- removed the C18 at (121.7, 59.8)
- removed the C18 at (162.2, 59.8)
- removed the C18 at (162.2, 31.8)
- removed the C18 at (121.7, 31.8)
- removed the C18 at (121.7, 87.8)
- removed the C2 at (120.8, 66.2)
- removed the C2 at (161.3, 38.1)
- removed the C2 at (161.3, 66.2)
- removed the C2 at (120.8, 38.1)
- removed the C2 at (161.3, 94.2)
- removed the C2 at (120.8, 94.2)
- removed the C3 at (168.2, 71.6)
- removed the C3 at (168.2, 99.6)
- removed the C3 at (127.6, 71.6)
- removed the C3 at (127.6, 99.6)
- removed the C3 at (127.6, 43.6)
- removed the C3 at (168.2, 43.6)
- removed the C4 at (170.9, 67.1)
- removed the C4 at (170.9, 95.1)
- removed the C4 at (130.3, 39.1)
- removed the C4 at (130.3, 95.1)
- removed the C4 at (130.3, 67.1)
- removed the C4 at (170.9, 39.1)
- removed the C5 at (162.9, 43.6)
- removed the C5 at (162.9, 71.6)
- removed the C5 at (122.3, 99.6)
- removed the C5 at (162.9, 99.6)
- removed the C5 at (122.3, 71.6)
- removed the C5 at (122.3, 43.6)
- removed the C6 at (160.4, 43.9)
- removed the C6 at (119.8, 71.9)
- removed the C6 at (160.4, 71.9)
- removed the C6 at (119.8, 99.9)
- removed the C6 at (119.8, 43.9)
- removed the C6 at (160.4, 99.9)
- removed the C7 at (122.0, 34.2)
- removed the C7 at (122.0, 62.2)
- removed the C7 at (162.6, 90.2)
- removed the C7 at (122.0, 90.2)
- removed the C7 at (162.6, 62.2)
- removed the C7 at (162.6, 34.2)
- removed the C8 at (131.7, 66.2)
- removed the C8 at (172.3, 38.2)
- removed the C8 at (131.7, 38.2)
- removed the C8 at (172.3, 94.2)
- removed the C8 at (131.7, 94.2)
- removed the C8 at (172.3, 66.2)
- removed the C9 at (175.3, 66.2)
- removed the C9 at (134.7, 94.2)
- removed the C9 at (175.3, 94.2)
- removed the C9 at (175.3, 38.2)
- removed the C9 at (134.7, 66.2)
- removed the C9 at (134.7, 38.2)
- removed the D1 at (169.8, 104.0)
- removed the D1 at (169.8, 76.0)
- removed the D1 at (129.2, 76.0)
- removed the D1 at (169.8, 48.0)
- removed the D1 at (129.2, 104.0)
- removed the D1 at (129.2, 48.0)
- removed the FID1 at (117.9, 84.0)
- removed the FID1 at (158.5, 28.0)
- removed the FID1 at (158.5, 84.0)
- removed the FID1 at (158.5, 56.0)
- removed the FID1 at (117.9, 56.0)
- removed the FID1 at (117.9, 28.0)
- removed the FID2 at (158.5, 70.5)
- removed the FID2 at (117.9, 98.5)
- removed the FID2 at (117.9, 70.5)
- removed the FID2 at (117.9, 42.5)
- removed the FID2 at (158.5, 42.5)
- removed the FID2 at (158.5, 98.5)
- removed the FID3 at (133.4, 56.0)
- removed the FID3 at (133.4, 84.0)
- removed the FID3 at (174.0, 84.0)
- removed the FID3 at (133.4, 28.0)
- removed the FID3 at (174.0, 28.0)
- removed the FID3 at (174.0, 56.0)
- removed the FLT1 at (136.6, 65.7)
- removed the FLT1 at (136.6, 93.7)
- removed the FLT1 at (177.2, 93.7)
- removed the FLT1 at (177.2, 37.7)
- removed the FLT1 at (136.6, 37.7)
- removed the FLT1 at (177.2, 65.7)
- removed the H2 at (177.0, 106.0)
- removed the H2 at (136.4, 106.0)
- removed the H2 at (177.0, 78.0)
- removed the H2 at (136.4, 78.0)
- removed the H2 at (136.4, 50.0)
- removed the H2 at (177.0, 50.0)
- removed the H3 at (119.2, 105.8)
- removed the H3 at (159.8, 105.8)
- removed the H3 at (159.8, 49.8)
- removed the H3 at (119.2, 77.8)
- removed the H3 at (119.2, 49.8)
- removed the H3 at (159.8, 77.8)
- removed the H4 at (136.4, 85.0)
- removed the H4 at (136.4, 57.0)
- removed the H4 at (177.0, 85.0)
- removed the H4 at (177.0, 29.0)
- removed the H4 at (177.0, 57.0)
- removed the H4 at (136.4, 29.0)
- removed the J1 at (112.4, 87.0)
- removed the J1 at (153.0, 59.0)
- removed the J1 at (112.4, 31.0)
- removed the J1 at (153.0, 87.0)
- removed the J1 at (153.0, 31.0)
- removed the J1 at (112.4, 59.0)
- removed the J3 at (129.0, 78.6)
- removed the J3 at (169.6, 78.6)
- removed the J3 at (129.0, 50.6)
- removed the J3 at (169.6, 106.6)
- removed the J3 at (129.0, 106.6)
- removed the J3 at (169.6, 50.6)
- removed KiKit_FID_B_1, KiKit_FID_B_2, KiKit_FID_B_3, KiKit_FID_T_1, KiKit_FID_T_2, KiKit_FID_T_3: Fiducial, Fiducial
- removed the L1 at (173.8, 65.7)
- removed the L1 at (173.8, 93.7)
- removed the L1 at (133.2, 37.7)
- removed the L1 at (133.2, 93.7)
- removed the L1 at (173.8, 37.7)
- removed the L1 at (133.2, 65.7)
- removed the L2 at (164.9, 33.1)
- removed the L2 at (124.3, 61.1)
- removed the L2 at (164.9, 89.1)
- removed the L2 at (124.3, 33.1)
- removed the L2 at (124.3, 89.1)
- removed the L2 at (164.9, 61.1)
- removed the L3 at (125.3, 59.2)
- removed the L3 at (165.9, 59.2)
- removed the L3 at (125.3, 31.2)
- removed the L3 at (165.9, 31.2)
- removed the L3 at (165.9, 87.2)
- removed the L3 at (125.3, 87.2)
- removed the Q1 at (177.2, 45.8)
- removed the Q1 at (136.6, 73.8)
- removed the Q1 at (136.6, 45.8)
- removed the Q1 at (177.2, 73.8)
- removed the Q1 at (136.6, 101.8)
- removed the Q1 at (177.2, 101.8)
- removed the R1 at (155.8, 69.1)
- removed the R1 at (155.8, 41.1)
- removed the R1 at (115.2, 69.1)
- removed the R1 at (155.8, 97.1)
- removed the R1 at (115.2, 97.1)
- removed the R1 at (115.2, 41.1)
- removed the R2 at (113.3, 41.1)
- removed the R2 at (153.9, 41.1)
- removed the R2 at (153.9, 97.1)
- removed the R2 at (153.9, 69.1)
- removed the R2 at (113.3, 97.1)
- removed the R2 at (113.3, 69.1)
- removed the R3 at (133.0, 77.6)
- removed the R3 at (173.6, 49.6)
- removed the R3 at (133.0, 49.6)
- removed the R3 at (133.0, 105.6)
- removed the R3 at (173.6, 105.6)
- removed the R3 at (173.6, 77.6)
- removed the R4 at (175.8, 43.6)
- removed the R4 at (135.2, 43.6)
- removed the R4 at (175.8, 99.6)
- removed the R4 at (175.8, 71.6)
- removed the R4 at (135.2, 99.6)
- removed the R4 at (135.2, 71.6)
- removed the RST1 at (114.5, 47.8)
- removed the RST1 at (155.1, 103.8)
- removed the RST1 at (155.1, 75.8)
- removed the RST1 at (114.5, 75.8)
- removed the RST1 at (114.5, 103.8)
- removed the RST1 at (155.1, 47.8)
- removed the U1 at (166.2, 38.9)
- removed the U1 at (166.2, 66.9)
- removed the U1 at (166.2, 94.9)
- removed the U1 at (125.5, 94.9)
- removed the U1 at (125.5, 38.9)
- removed the U1 at (125.5, 66.9)
- removed the U2 at (114.2, 66.7)
- removed the U2 at (114.2, 38.7)
- removed the U2 at (154.8, 66.7)
- removed the U2 at (154.8, 38.7)
- removed the U2 at (114.2, 94.7)
- removed the U2 at (154.8, 94.7)
- removed the Y1 at (131.0, 88.3)
- removed the Y1 at (131.0, 60.3)
- removed the Y1 at (131.0, 32.3)
- removed the Y1 at (171.6, 88.3)
- removed the Y1 at (171.6, 60.3)
- removed the Y1 at (171.6, 32.3)
- removed the Y2 at (165.3, 72.3)
- removed the Y2 at (124.7, 72.3)
- removed the Y2 at (124.7, 44.3)
- removed the Y2 at (124.7, 100.3)
- removed the Y2 at (165.3, 44.3)
- removed the Y2 at (165.3, 100.3)
- added AE1: Antenna, RF_Antenna:Texas_SWRA117D_2.4GHz_Right, F.Cu at (180.8, 63.9)
- added AE1: Antenna, RF_Antenna:Texas_SWRA117D_2.4GHz_Right, F.Cu at (140.2, 35.9)
- added AE1: Antenna, RF_Antenna:Texas_SWRA117D_2.4GHz_Right, F.Cu at (140.2, 63.9)
- added AE1: Antenna, RF_Antenna:Texas_SWRA117D_2.4GHz_Right, F.Cu at (180.8, 35.9)
- added BT1: Battery_Cell, Battery:BatteryHolder_MPD_BC2003_1x2032, B.Cu at (165.9, 40.6)
- added BT1: Battery_Cell, Battery:BatteryHolder_MPD_BC2003_1x2032, B.Cu at (125.3, 40.6)
- added BT1: Battery_Cell, Battery:BatteryHolder_MPD_BC2003_1x2032, B.Cu at (165.9, 68.6)
- added BT1: Battery_Cell, Battery:BatteryHolder_MPD_BC2003_1x2032, B.Cu at (125.3, 68.6)
- added C1: 100n, Capacitor_SMD:C_0402_1005Metric, F.Cu at (161.2, 71.2)
- added C1: 100n, Capacitor_SMD:C_0402_1005Metric, F.Cu at (161.2, 43.2)
- added C1: 100n, Capacitor_SMD:C_0402_1005Metric, F.Cu at (120.5, 71.2)
- added C1: 100n, Capacitor_SMD:C_0402_1005Metric, F.Cu at (120.5, 43.2)
- added C10: 100p, Capacitor_SMD:C_0402_1005Metric, F.Cu at (130.3, 64.5)
- added C10: 100p, Capacitor_SMD:C_0402_1005Metric, F.Cu at (170.9, 64.5)
- added C10: 100p, Capacitor_SMD:C_0402_1005Metric, F.Cu at (130.3, 36.5)
- added C10: 100p, Capacitor_SMD:C_0402_1005Metric, F.Cu at (170.9, 36.5)
- added C11: 100n, Capacitor_SMD:C_0402_1005Metric, F.Cu at (171.9, 64.5)
- added C11: 100n, Capacitor_SMD:C_0402_1005Metric, F.Cu at (131.3, 36.5)
- added C11: 100n, Capacitor_SMD:C_0402_1005Metric, F.Cu at (171.9, 36.5)
- added C11: 100n, Capacitor_SMD:C_0402_1005Metric, F.Cu at (131.3, 64.5)
- added C12: 100n, Capacitor_SMD:C_0402_1005Metric, F.Cu at (152.8, 39.6)
- added C12: 100n, Capacitor_SMD:C_0402_1005Metric, F.Cu at (112.2, 67.6)
- added C12: 100n, Capacitor_SMD:C_0402_1005Metric, F.Cu at (112.2, 39.6)
- added C12: 100n, Capacitor_SMD:C_0402_1005Metric, F.Cu at (152.8, 67.6)
- added C13: 100n, Capacitor_SMD:C_0402_1005Metric, F.Cu at (168.2, 73.7)
- added C13: 100n, Capacitor_SMD:C_0402_1005Metric, F.Cu at (127.6, 45.7)
- added C13: 100n, Capacitor_SMD:C_0402_1005Metric, F.Cu at (168.2, 45.7)
- added C13: 100n, Capacitor_SMD:C_0402_1005Metric, F.Cu at (127.6, 73.7)
- added C14: 10p, Capacitor_SMD:C_0402_1005Metric, F.Cu at (164.1, 74.8)
- added C14: 10p, Capacitor_SMD:C_0402_1005Metric, F.Cu at (164.1, 46.8)
- added C14: 10p, Capacitor_SMD:C_0402_1005Metric, F.Cu at (123.5, 74.8)
- added C14: 10p, Capacitor_SMD:C_0402_1005Metric, F.Cu at (123.5, 46.8)
- added C15: 10p, Capacitor_SMD:C_0402_1005Metric, F.Cu at (166.4, 74.8)
- added C15: 10p, Capacitor_SMD:C_0402_1005Metric, F.Cu at (125.8, 74.8)
- added C15: 10p, Capacitor_SMD:C_0402_1005Metric, F.Cu at (166.4, 46.8)
- added C15: 10p, Capacitor_SMD:C_0402_1005Metric, F.Cu at (125.8, 46.8)
- added C16: 4u7, Capacitor_SMD:C_0603_1608Metric, F.Cu at (126.4, 34.7)
- added C16: 4u7, Capacitor_SMD:C_0603_1608Metric, F.Cu at (167.0, 62.7)
- added C16: 4u7, Capacitor_SMD:C_0603_1608Metric, F.Cu at (167.0, 34.7)
- added C16: 4u7, Capacitor_SMD:C_0603_1608Metric, F.Cu at (126.4, 62.7)
- added C17: 100n, Capacitor_SMD:C_0402_1005Metric, F.Cu at (121.9, 34.1)
- added C17: 100n, Capacitor_SMD:C_0402_1005Metric, F.Cu at (162.5, 62.1)
- added C17: 100n, Capacitor_SMD:C_0402_1005Metric, F.Cu at (121.9, 62.1)
- added C17: 100n, Capacitor_SMD:C_0402_1005Metric, F.Cu at (162.5, 34.1)
- added C18: 4u7, Capacitor_SMD:C_0603_1608Metric, F.Cu at (162.2, 32.8)
- added C18: 4u7, Capacitor_SMD:C_0603_1608Metric, F.Cu at (121.7, 32.8)
- added C18: 4u7, Capacitor_SMD:C_0603_1608Metric, F.Cu at (121.7, 60.8)
- added C18: 4u7, Capacitor_SMD:C_0603_1608Metric, F.Cu at (162.2, 60.8)
- added C2: 100n, Capacitor_SMD:C_0402_1005Metric, F.Cu at (161.3, 67.2)
- added C2: 100n, Capacitor_SMD:C_0402_1005Metric, F.Cu at (120.8, 39.2)
- added C2: 100n, Capacitor_SMD:C_0402_1005Metric, F.Cu at (161.3, 39.2)
- added C2: 100n, Capacitor_SMD:C_0402_1005Metric, F.Cu at (120.8, 67.2)
- added C3: 100n, Capacitor_SMD:C_0402_1005Metric, F.Cu at (168.2, 72.6)
- added C3: 100n, Capacitor_SMD:C_0402_1005Metric, F.Cu at (127.6, 44.6)
- added C3: 100n, Capacitor_SMD:C_0402_1005Metric, F.Cu at (168.2, 44.6)
- added C3: 100n, Capacitor_SMD:C_0402_1005Metric, F.Cu at (127.6, 72.6)
- added C4: 100n, Capacitor_SMD:C_0402_1005Metric, F.Cu at (170.9, 68.1)
- added C4: 100n, Capacitor_SMD:C_0402_1005Metric, F.Cu at (170.9, 40.1)
- added C4: 100n, Capacitor_SMD:C_0402_1005Metric, F.Cu at (130.3, 40.1)
- added C4: 100n, Capacitor_SMD:C_0402_1005Metric, F.Cu at (130.3, 68.1)
- added C5: 100n, Capacitor_SMD:C_0402_1005Metric, F.Cu at (162.9, 72.6)
- added C5: 100n, Capacitor_SMD:C_0402_1005Metric, F.Cu at (122.3, 44.6)
- added C5: 100n, Capacitor_SMD:C_0402_1005Metric, F.Cu at (162.9, 44.6)
- added C5: 100n, Capacitor_SMD:C_0402_1005Metric, F.Cu at (122.3, 72.6)
- added C6: 4u7, Capacitor_SMD:C_0603_1608Metric, F.Cu at (119.8, 72.9)
- added C6: 4u7, Capacitor_SMD:C_0603_1608Metric, F.Cu at (160.4, 72.9)
- added C6: 4u7, Capacitor_SMD:C_0603_1608Metric, F.Cu at (160.4, 44.9)
- added C6: 4u7, Capacitor_SMD:C_0603_1608Metric, F.Cu at (119.8, 44.9)
- added C7: 100n, Capacitor_SMD:C_0402_1005Metric, F.Cu at (122.0, 63.2)
- added C7: 100n, Capacitor_SMD:C_0402_1005Metric, F.Cu at (122.0, 35.2)
- added C7: 100n, Capacitor_SMD:C_0402_1005Metric, F.Cu at (162.6, 63.2)
- added C7: 100n, Capacitor_SMD:C_0402_1005Metric, F.Cu at (162.6, 35.2)
- added C8: 0p8, Capacitor_SMD:C_0402_1005Metric, F.Cu at (172.3, 39.2)
- added C8: 0p8, Capacitor_SMD:C_0402_1005Metric, F.Cu at (131.7, 67.2)
- added C8: 0p8, Capacitor_SMD:C_0402_1005Metric, F.Cu at (172.3, 67.2)
- added C8: 0p8, Capacitor_SMD:C_0402_1005Metric, F.Cu at (131.7, 39.2)
- added C9: 0p3, Capacitor_SMD:C_0402_1005Metric, F.Cu at (175.3, 39.2)
- added C9: 0p3, Capacitor_SMD:C_0402_1005Metric, F.Cu at (175.3, 67.2)
- added C9: 0p3, Capacitor_SMD:C_0402_1005Metric, F.Cu at (134.7, 39.2)
- added C9: 0p3, Capacitor_SMD:C_0402_1005Metric, F.Cu at (134.7, 67.2)
- added D1: LED, LED_SMD:LED_0603_1608Metric, F.Cu at (169.8, 77.0)
- added D1: LED, LED_SMD:LED_0603_1608Metric, F.Cu at (129.2, 77.0)
- added D1: LED, LED_SMD:LED_0603_1608Metric, F.Cu at (169.8, 49.0)
- added D1: LED, LED_SMD:LED_0603_1608Metric, F.Cu at (129.2, 49.0)
- added FID1: Fiducial, Fiducial:Fiducial_0.5mm_Mask1mm, F.Cu at (174.0, 80.0)
- added FID1: Fiducial, Fiducial:Fiducial_0.5mm_Mask1mm, F.Cu at (174.0, 52.0)
- added FID1: Fiducial, Fiducial:Fiducial_0.5mm_Mask1mm, F.Cu at (133.4, 80.0)
- added FID1: Fiducial, Fiducial:Fiducial_0.5mm_Mask1mm, F.Cu at (133.4, 52.0)
- added FID2: Fiducial, Fiducial:Fiducial_0.5mm_Mask1mm, F.Cu at (110.4, 52.0)
- added FID2: Fiducial, Fiducial:Fiducial_0.5mm_Mask1mm, F.Cu at (151.0, 52.0)
- added FID2: Fiducial, Fiducial:Fiducial_0.5mm_Mask1mm, F.Cu at (151.0, 80.0)
- added FID2: Fiducial, Fiducial:Fiducial_0.5mm_Mask1mm, F.Cu at (110.4, 80.0)
- added FID3: Fiducial, Fiducial:Fiducial_0.5mm_Mask1mm, F.Cu at (174.0, 29.0)
- added FID3: Fiducial, Fiducial:Fiducial_0.5mm_Mask1mm, F.Cu at (174.0, 57.0)
- added FID3: Fiducial, Fiducial:Fiducial_0.5mm_Mask1mm, F.Cu at (133.4, 29.0)
- added FID3: Fiducial, Fiducial:Fiducial_0.5mm_Mask1mm, F.Cu at (133.4, 57.0)
- added FLT1: DLF162500LT-5028A1, DLF162500:DLF162500LT-5028A1, F.Cu at (177.2, 38.7)
- added FLT1: DLF162500LT-5028A1, DLF162500:DLF162500LT-5028A1, F.Cu at (136.6, 66.7)
- added FLT1: DLF162500LT-5028A1, DLF162500:DLF162500LT-5028A1, F.Cu at (177.2, 66.7)
- added FLT1: DLF162500LT-5028A1, DLF162500:DLF162500LT-5028A1, F.Cu at (136.6, 38.7)
- added H2: MountingHole, MountingHole:MountingHole_2.2mm_M2_DIN965, F.Cu at (136.4, 51.0)
- added H2: MountingHole, MountingHole:MountingHole_2.2mm_M2_DIN965, F.Cu at (177.0, 51.0)
- added H2: MountingHole, MountingHole:MountingHole_2.2mm_M2_DIN965, F.Cu at (136.4, 79.0)
- added H2: MountingHole, MountingHole:MountingHole_2.2mm_M2_DIN965, F.Cu at (177.0, 79.0)
- added H3: MountingHole, MountingHole:MountingHole_2.2mm_M2_DIN965, F.Cu at (119.2, 50.8)
- added H3: MountingHole, MountingHole:MountingHole_2.2mm_M2_DIN965, F.Cu at (119.2, 78.8)
- added H3: MountingHole, MountingHole:MountingHole_2.2mm_M2_DIN965, F.Cu at (159.8, 78.8)
- added H3: MountingHole, MountingHole:MountingHole_2.2mm_M2_DIN965, F.Cu at (159.8, 50.8)
- added H4: MountingHole, MountingHole:MountingHole_2.2mm_M2_DIN965, F.Cu at (177.0, 30.0)
- added H4: MountingHole, MountingHole:MountingHole_2.2mm_M2_DIN965, F.Cu at (177.0, 58.0)
- added H4: MountingHole, MountingHole:MountingHole_2.2mm_M2_DIN965, F.Cu at (136.4, 30.0)
- added H4: MountingHole, MountingHole:MountingHole_2.2mm_M2_DIN965, F.Cu at (136.4, 58.0)
- added J1: Conn_ARM_SWD_TagConnect_TC2030, Connector:Tag-Connect_TC2030-IDC-NL_2x03_P1.27mm_Vertical, F.Cu at (112.4, 60.0)
- added J1: Conn_ARM_SWD_TagConnect_TC2030, Connector:Tag-Connect_TC2030-IDC-NL_2x03_P1.27mm_Vertical, F.Cu at (153.0, 32.0)
- added J1: Conn_ARM_SWD_TagConnect_TC2030, Connector:Tag-Connect_TC2030-IDC-NL_2x03_P1.27mm_Vertical, F.Cu at (153.0, 60.0)
- added J1: Conn_ARM_SWD_TagConnect_TC2030, Connector:Tag-Connect_TC2030-IDC-NL_2x03_P1.27mm_Vertical, F.Cu at (112.4, 32.0)
- added J3: ~, Connector_PinHeader_2.00mm:PinHeader_1x04_P2.00mm_Vertical, F.Cu at (169.6, 79.6)
- added J3: ~, Connector_PinHeader_2.00mm:PinHeader_1x04_P2.00mm_Vertical, F.Cu at (129.0, 79.6)
- added J3: ~, Connector_PinHeader_2.00mm:PinHeader_1x04_P2.00mm_Vertical, F.Cu at (129.0, 51.6)
- added J3: ~, Connector_PinHeader_2.00mm:PinHeader_1x04_P2.00mm_Vertical, F.Cu at (169.6, 51.6)
- added L1: 2nH7, Inductor_SMD:L_0402_1005Metric, F.Cu at (173.8, 66.7)
- added L1: 2nH7, Inductor_SMD:L_0402_1005Metric, F.Cu at (133.2, 38.7)
- added L1: 2nH7, Inductor_SMD:L_0402_1005Metric, F.Cu at (133.2, 66.7)
- added L1: 2nH7, Inductor_SMD:L_0402_1005Metric, F.Cu at (173.8, 38.7)
- added L2: 10nH, Inductor_SMD:L_0402_1005Metric, F.Cu at (124.3, 62.1)
- added L2: 10nH, Inductor_SMD:L_0402_1005Metric, F.Cu at (164.9, 34.1)
- added L2: 10nH, Inductor_SMD:L_0402_1005Metric, F.Cu at (124.3, 34.1)
- added L2: 10nH, Inductor_SMD:L_0402_1005Metric, F.Cu at (164.9, 62.1)
- added L3: 10uH, Inductor_SMD:L_0805_2012Metric, F.Cu at (165.9, 60.2)
- added L3: 10uH, Inductor_SMD:L_0805_2012Metric, F.Cu at (125.3, 32.2)
- added L3: 10uH, Inductor_SMD:L_0805_2012Metric, F.Cu at (125.3, 60.2)
- added L3: 10uH, Inductor_SMD:L_0805_2012Metric, F.Cu at (165.9, 32.2)
- added Q1: Q_Photo_NPN, Diode_SMD:D_0603_1608Metric, F.Cu at (136.6, 46.8)
- added Q1: Q_Photo_NPN, Diode_SMD:D_0603_1608Metric, F.Cu at (177.2, 74.8)
- added Q1: Q_Photo_NPN, Diode_SMD:D_0603_1608Metric, F.Cu at (177.2, 46.8)
- added Q1: Q_Photo_NPN, Diode_SMD:D_0603_1608Metric, F.Cu at (136.6, 74.8)
- added R1: 10k, Resistor_SMD:R_0402_1005Metric, F.Cu at (157.4, 40.7)
- added R1: 10k, Resistor_SMD:R_0402_1005Metric, F.Cu at (116.8, 40.7)
- added R1: 10k, Resistor_SMD:R_0402_1005Metric, F.Cu at (116.8, 68.7)
- added R1: 10k, Resistor_SMD:R_0402_1005Metric, F.Cu at (157.4, 68.7)
- added R2: 10k, Resistor_SMD:R_0402_1005Metric, F.Cu at (116.8, 66.5)
- added R2: 10k, Resistor_SMD:R_0402_1005Metric, F.Cu at (157.4, 38.5)
- added R2: 10k, Resistor_SMD:R_0402_1005Metric, F.Cu at (116.8, 38.5)
- added R2: 10k, Resistor_SMD:R_0402_1005Metric, F.Cu at (157.4, 66.5)
- added R3: 1k, Resistor_SMD:R_0402_1005Metric, F.Cu at (133.0, 78.0)
- added R3: 1k, Resistor_SMD:R_0402_1005Metric, F.Cu at (173.6, 78.0)
- added R3: 1k, Resistor_SMD:R_0402_1005Metric, F.Cu at (173.6, 50.0)
- added R3: 1k, Resistor_SMD:R_0402_1005Metric, F.Cu at (133.0, 50.0)
- added R4: 470, Resistor_SMD:R_0402_1005Metric, F.Cu at (175.8, 72.6)
- added R4: 470, Resistor_SMD:R_0402_1005Metric, F.Cu at (135.2, 72.6)
- added R4: 470, Resistor_SMD:R_0402_1005Metric, F.Cu at (135.2, 44.6)
- added R4: 470, Resistor_SMD:R_0402_1005Metric, F.Cu at (175.8, 44.6)
- added RST1: B3U-1000P, Button_Switch_SMD:SW_SPST_B3U-1000P, F.Cu at (155.1, 76.8)
- added RST1: B3U-1000P, Button_Switch_SMD:SW_SPST_B3U-1000P, F.Cu at (114.5, 48.8)
- added RST1: B3U-1000P, Button_Switch_SMD:SW_SPST_B3U-1000P, F.Cu at (155.1, 48.8)
- added RST1: B3U-1000P, Button_Switch_SMD:SW_SPST_B3U-1000P, F.Cu at (114.5, 76.8)
- added U1: STM32WB55CGUx, Package_DFN_QFN:QFN-48-1EP_7x7mm_P0.5mm_EP5.6x5.6mm, F.Cu at (166.2, 67.9)
- added U1: STM32WB55CGUx, Package_DFN_QFN:QFN-48-1EP_7x7mm_P0.5mm_EP5.6x5.6mm, F.Cu at (125.5, 67.9)
- added U1: STM32WB55CGUx, Package_DFN_QFN:QFN-48-1EP_7x7mm_P0.5mm_EP5.6x5.6mm, F.Cu at (166.2, 39.9)
- added U1: STM32WB55CGUx, Package_DFN_QFN:QFN-48-1EP_7x7mm_P0.5mm_EP5.6x5.6mm, F.Cu at (125.5, 39.9)
- added U2: SHT4x, Sensor_Humidity:Sensirion_DFN-4_1.5x1.5mm_P0.8mm_SHT4x_NoCentralPad, F.Cu at (114.2, 67.6)
- added U2: SHT4x, Sensor_Humidity:Sensirion_DFN-4_1.5x1.5mm_P0.8mm_SHT4x_NoCentralPad, F.Cu at (154.8, 39.6)
- added U2: SHT4x, Sensor_Humidity:Sensirion_DFN-4_1.5x1.5mm_P0.8mm_SHT4x_NoCentralPad, F.Cu at (154.8, 67.6)
- added U2: SHT4x, Sensor_Humidity:Sensirion_DFN-4_1.5x1.5mm_P0.8mm_SHT4x_NoCentralPad, F.Cu at (114.2, 39.6)
- added Y1: 32 MHz, Crystal:Crystal_SMD_2016-4Pin_2.0x1.6mm, F.Cu at (171.6, 61.3)
- added Y1: 32 MHz, Crystal:Crystal_SMD_2016-4Pin_2.0x1.6mm, F.Cu at (131.0, 61.3)
- added Y1: 32 MHz, Crystal:Crystal_SMD_2016-4Pin_2.0x1.6mm, F.Cu at (171.6, 33.3)
- added Y1: 32 MHz, Crystal:Crystal_SMD_2016-4Pin_2.0x1.6mm, F.Cu at (131.0, 33.3)
- added Y2: 32.768KHz, Crystal:Crystal_SMD_2012-2Pin_2.0x1.2mm, F.Cu at (124.7, 45.3)
- added Y2: 32.768KHz, Crystal:Crystal_SMD_2012-2Pin_2.0x1.2mm, F.Cu at (165.3, 73.3)
- added Y2: 32.768KHz, Crystal:Crystal_SMD_2012-2Pin_2.0x1.2mm, F.Cu at (165.3, 45.3)
- added Y2: 32.768KHz, Crystal:Crystal_SMD_2012-2Pin_2.0x1.2mm, F.Cu at (124.7, 73.3)
Routing:
- net Board_5-+3.3V: track 67.1 -> 0.00 mm, vias 12 -> 0
- net Board_4-+3.3V: track 67.1 -> 0.00 mm, vias 12 -> 0
- net Board_4-/NRST: track 38.9 -> 0.00 mm
- net Board_5-/NRST: track 38.9 -> 0.00 mm
- net Board_4-/UART_RX: track 29.1 -> 0.00 mm, vias 1 -> 0
- net Board_5-/UART_RX: track 29.1 -> 0.00 mm, vias 1 -> 0
- net Board_5-/UART_TX: track 17.3 -> 0.00 mm, vias 1 -> 0
- net Board_4-/UART_TX: track 17.3 -> 0.00 mm, vias 1 -> 0
- net Board_4-SCL: track 17.3 -> 0.00 mm
- net Board_5-SCL: track 17.3 -> 0.00 mm
- net Board_5-SWDCLK: track 14.4 -> 0.00 mm
- net Board_4-SWDCLK: track 14.4 -> 0.00 mm
- net Board_4-GND: track 12.7 -> 0.00 mm, vias 100 -> 0
- net Board_5-GND: track 12.7 -> 0.00 mm, vias 100 -> 0
- net Board_5-SWDIO: track 12.7 -> 0.00 mm
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- removed copper zone on B.Cu, net Board_4-+3.3V
- removed copper zone on F.Cu, net Board_4-/VFBSMPS
- removed copper zone on F.Cu, net Board_4-GND
- removed copper zone on In1.Cu, net Board_4-GND
- removed copper zone on In2.Cu, net Board_4-GND
- removed copper zone on B.Cu, net Board_5-+3.3V
- removed copper zone on F.Cu, net Board_5-/VFBSMPS
- removed copper zone on F.Cu, net Board_5-GND
- removed copper zone on In1.Cu, net Board_5-GND
- removed copper zone on In2.Cu, net Board_5-GND
Other:
- board size 92.2 x 95 mm -> 78.2 x 69 mm
- board text added: "0.4"
- board text removed: "0.2"
